Commit message: Imported upstream version '0.1.0' of 'upstream'

File: scitos_description/urdf/scitos.xacro (robot description, xacro)
@@ -353,63 +353,3 @@
     <child link="head_xtion_rgb_optical_frame"/>
   </joint>
-  <!-- Connect base to chest_xtion_link -->
-  <link name="chest_xtion_link">
-    <visual>
-      <origin rpy="3.14 0 0" xyz="0 0 0"/>
-      <geometry>
-        <mesh filename="package://scitos_description/meshes/xtion.dae"/>
-      </geometry>
-    </visual>
-    <collision>
-      <origin rpy="0 0 0" xyz="0 0 0.071"/>
-      <geometry>
-        <box size="0.001 0.001 0.001"/>
-      </geometry>
-    </collision>
-  </link>
-  <link name="chest_xtion_height_tilt_link"/>
-  <joint name="chest_xtion_height_joint" type="prismatic" >
-    <!-- Z height from calibrate_chest -->
-    <axis xyz="0 0 1"/>
-    <origin rpy="0 0 0" xyz="0.12 0 0" />
-    <limit effort="1000" velocity="1000" lower="0.5" upper="1.5"/>
-    <parent link="base_link"/>
-    <child link="chest_xtion_height_tilt_link"/>
-  </joint>
-  <joint name="chest_xtion_tilt_joint" type="continuous" >
-    <!-- Rotation y angle from calibrate_chest-->
-    <axis xyz="0 1 0"/>
-    <origin rpy="0 0 0" xyz="0 0 0" />
-    <parent link="chest_xtion_height_tilt_link"/>
-    <child link="chest_xtion_link"/>
-  </joint>
-  <!-- chest_xtion internal frames -->
-  <link name="chest_xtion_depth_frame"/>
-  <link name="chest_xtion_rgb_frame"/>
-  <link name="chest_xtion_depth_optical_frame"/>
-  <link name="chest_xtion_rgb_optical_frame"/>
-  <joint name="chest_xtion_base_link" type="fixed" >
-    <origin rpy="0 0 0"
-            xyz="0 0.045 0" />
-    <parent link="chest_xtion_link"/>
-    <child link="chest_xtion_depth_frame"/>
-  </joint>
-  <joint name="chest_xtion_base_link1" type="fixed" >
-    <origin rpy="0 0 0"
-            xyz="0 0.02 0" />
-    <parent link="chest_xtion_link"/>
-    <child link="chest_xtion_rgb_frame"/>
-  </joint>
-  <joint name="chest_xtion_base_link2" type="fixed" >
-    <origin rpy="-1.5707963267948966 0 -1.5707963267948966"
-            xyz="0 0 0" />
-    <parent link="chest_xtion_depth_frame"/>
-    <child link="chest_xtion_depth_optical_frame"/>
-  </joint>
-  <joint name="chest_xtion_base_link3" type="fixed" >
-    <origin rpy="-1.5707963267948966 0 -1.5707963267948966"
-            xyz="0 0 0" />
-    <parent link="chest_xtion_rgb_frame"/>
-    <child link="chest_xtion_rgb_optical_frame"/>
-  </joint>
 </robot>
